File: LuMini_3Inch.sch (EAGLE design)
At the start: 79 parts, among them J1 SOLDER_PAD_2, J2 SOLDER_PAD_2, J3 SOLDER_PAD_2

Commit message: added lumini ring
Parts:
- removed D1, D10, D11, D12, D13, D14, D15, D16, D17, D18, D19, D2, D20, D21, D22, D23, D24, D25, D26, D27, D28, D29, D3, D30, D31, D32, D33, D34, D35, D36, D37, D38, D39, D4, D40, D41, D42, D43, D44, D45, D46, D47, D48, D49, D5, D50, D51, D52, D53, D54, D55, D56, D57, D58, D59, D6, D60, D7, D8, D9: APA102-2020, SparkFun-LED:APA102-2020
Connections:
- removed net N$1: D4.CO, D5.CI
- removed net N$10: D4.DO, D5.DI
- removed net N$100: D50.CO, D51.CI
- removed net N$101: D50.DO, D51.DI
- removed net N$102: D51.CO, D52.CI
- removed net N$103: D51.DO, D52.DI
- removed net N$104: D52.CO, D53.CI
- removed net N$105: D52.DO, D53.DI
- removed net N$106: D53.CO, D54.CI
- removed net N$107: D53.DO, D54.DI
- removed net N$108: D54.CO, D55.CI
- removed net N$109: D54.DO, D55.DI
- removed net N$11: D5.CO, D6.CI
- removed net N$110: D55.CO, D56.CI
- removed net N$111: D55.DO, D56.DI
- removed net N$112: D57.CO, D58.CI
- removed net N$113: D57.DO, D58.DI
- removed net N$114: D58.DO, D59.DI
- removed net N$115: D59.CO, D60.CI
- removed net N$116: D59.DO, D60.DI
- removed net N$117: D58.CO, D59.CI
- removed net N$118: D48.CO, D49.CI
- removed net N$119: D48.DO, D49.DI
- removed net N$12: D5.DO, D6.DI
- removed net N$120: D56.DO, D57.DI
- removed net N$121: D56.CO, D57.CI
- removed net N$124: D20.CO, D21.CI
- removed net N$13: D6.CO, D7.CI
- removed net N$14: D6.DO, D7.DI
- removed net N$15: D7.CO, D8.CI
- removed net N$16: D7.DO, D8.DI
- removed net N$17: D16.DO, D17.DI
- removed net N$18: D20.DO, D21.DI
- removed net N$19: D10.CI, D9.CO
- removed net N$20: D10.DI, D9.DO
- removed net N$21: D10.CO, D11.CI
- removed net N$22: D10.DO, D11.DI
- removed net N$23: D11.CO, D12.CI
- removed net N$24: D11.DO, D12.DI
- removed net N$25: D12.CO, D13.CI
- removed net N$26: D12.DO, D13.DI
- removed net N$27: D13.CO, D14.CI
- removed net N$28: D13.DO, D14.DI
- removed net N$29: D14.CO, D15.CI
- removed net N$30: D14.DO, D15.DI
- removed net N$31: D45.CO, D46.CI
- removed net N$32: D30.CO, D31.CI
- removed net N$33: D8.CO, D9.CI
- removed net N$34: D8.DO, D9.DI
- removed net N$35: D17.CO, D18.CI
- removed net N$36: D17.DO, D18.DI
- removed net N$37: D18.CO, D19.CI
- removed net N$38: D18.DO, D19.DI
- removed net N$39: D19.CO, D20.CI
- removed net N$4: D1.CO, D2.CI
- removed net N$40: D19.DO, D20.DI
- removed net N$41: D30.DO, D31.DI
- removed net N$42: D15.CO, D16.CI
- removed net N$43: D16.CO, D17.CI
- removed net N$44: D21.CO, D22.CI
- removed net N$45: D21.DO, D22.DI
- removed net N$46: D22.CO, D23.CI
- removed net N$47: D22.DO, D23.DI
- removed net N$48: D23.CO, D24.CI
- removed net N$49: D23.DO, D24.DI
- removed net N$5: D1.DO, D2.DI
- removed net N$50: D24.CO, D25.CI
- removed net N$51: D24.DO, D25.DI
- removed net N$52: D25.CO, D26.CI
- removed net N$53: D25.DO, D26.DI
- removed net N$54: D26.CO, D27.CI
- removed net N$55: D26.DO, D27.DI
- removed net N$56: D27.CO, D28.CI
- removed net N$57: D27.DO, D28.DI
- removed net N$58: D29.CO, D30.CI
- removed net N$59: D29.DO, D30.DI
- removed net N$6: D2.CO, D3.CI
- removed net N$60: D15.DO, D16.DI
- removed net N$61: D45.DO, D46.DI
- removed net N$62: D31.CO, D32.CI
- removed net N$63: D31.DO, D32.DI
- removed net N$64: D32.CO, D33.CI
- removed net N$65: D32.DO, D33.DI
- removed net N$66: D33.CO, D34.CI
- removed net N$67: D33.DO, D34.DI
- removed net N$68: D34.CO, D35.CI
- removed net N$69: D34.DO, D35.DI
- removed net N$7: D2.DO, D3.DI
- removed net N$70: D35.CO, D36.CI
- removed net N$71: D35.DO, D36.DI
- removed net N$72: D37.CO, D38.CI
- removed net N$73: D37.DO, D38.DI
- removed net N$74: D38.DO, D39.DI
- removed net N$75: D39.CO, D40.CI
- removed net N$76: D39.DO, D40.DI
- removed net N$77: D38.CO, D39.CI
- removed net N$78: D28.CO, D29.CI
- removed net N$79: D28.DO, D29.DI
- removed net N$8: D3.CO, D4.CI
- removed net N$80: D36.DO, D37.DI
- removed net N$81: D36.CO, D37.CI
- removed net N$82: D40.CO, D41.CI
- removed net N$83: D40.DO, D41.DI
- removed net N$84: D41.CO, D42.CI
- removed net N$85: D41.DO, D42.DI
- removed net N$86: D42.CO, D43.CI
- removed net N$87: D42.DO, D43.DI
- removed net N$88: D43.CO, D44.CI
- removed net N$89: D43.DO, D44.DI
- removed net N$9: D3.DO, D4.DI
- removed net N$90: D44.CO, D45.CI
- removed net N$91: D44.DO, D45.DI
- removed net N$94: D46.CO, D47.CI
- removed net N$95: D46.DO, D47.DI
- removed net N$96: D47.CO, D48.CI
- removed net N$97: D47.DO, D48.DI
- removed net N$98: D49.CO, D50.CI
- removed net N$99: D49.DO, D50.DI
- net 5V: no longer D1.VCC, D10.VCC, D11.VCC, D12.VCC, D13.VCC, D14.VCC, D15.VCC, D16.VCC, D17.VCC, D18.VCC, D19.VCC, D2.VCC, D20.VCC, D21.VCC, D22.VCC, D23.VCC, D24.VCC, D25.VCC, D26.VCC, D27.VCC, D28.VCC, D29.VCC, D3.VCC, D30.VCC, D31.VCC, D32.VCC, D33.VCC, D34.VCC, D35.VCC, D36.VCC, D37.VCC, D38.VCC, D39.VCC, D4.VCC, D40.VCC, D41.VCC, D42.VCC, D43.VCC, D44.VCC, D45.VCC, D46.VCC, D47.VCC, D48.VCC, D49.VCC, D5.VCC, D50.VCC, D51.VCC, D52.VCC, D53.VCC, D54.VCC, D55.VCC, D56.VCC, D57.VCC, D58.VCC, D59.VCC, D6.VCC, D60.VCC, D7.VCC, D8.VCC, D9.VCC
- net CI: no longer D1.CI
- net CO: no longer D60.CO
- net DI: no longer D1.DI
- net DO: no longer D60.DO
- net GND: no longer D1.GND, D10.GND, D11.GND, D12.GND, D13.GND, D14.GND, D15.GND, D16.GND, D17.GND, D18.GND, D19.GND, D2.GND, D20.GND, D21.GND, D22.GND, D23.GND, D24.GND, D25.GND, D26.GND, D27.GND, D28.GND, D29.GND, D3.GND, D30.GND, D31.GND, D32.GND, D33.GND, D34.GND, D35.GND, D36.GND, D37.GND, D38.GND, D39.GND, D4.GND, D40.GND, D41.GND, D42.GND, D43.GND, D44.GND, D45.GND, D46.GND, D47.GND, D48.GND, D49.GND, D5.GND, D50.GND, D51.GND, D52.GND, D53.GND, D54.GND, D55.GND, D56.GND, D57.GND, D58.GND, D59.GND, D6.GND, D60.GND, D7.GND, D8.GND, D9.GND
Other:
- note removed: "LED's"
- note removed: "Vin: 3.0V-5.5V"

Commit message: about to repin IVL
Parts:
- added D1, D10, D11, D12, D13, D14, D15, D16, D17, D18, D19, D2, D20, D21, D22, D23, D24, D25, D26, D27, D28, D29, D3, D30, D31, D32, D33, D34, D35, D36, D37, D38, D39, D4, D40, D41, D42, D43, D44, D45, D46, D47, D48, D49, D5, D50, D51, D52, D53, D54, D55, D56, D57, D58, D59, D6, D60, D7, D8, D9: APA102-2020, SparkFun-LED:APA102-2020
Connections:
- new net N$1: D4.CO, D5.CI
- new net N$10: D4.DO, D5.DI
- new net N$100: D50.CO, D51.CI
- new net N$101: D50.DO, D51.DI
- new net N$102: D51.CO, D52.CI
- new net N$103: D51.DO, D52.DI
- new net N$104: D52.CO, D53.CI
- new net N$105: D52.DO, D53.DI
- new net N$106: D53.CO, D54.CI
- new net N$107: D53.DO, D54.DI
- new net N$108: D54.CO, D55.CI
- new net N$109: D54.DO, D55.DI
- new net N$11: D5.CO, D6.CI
- new net N$110: D55.CO, D56.CI
- new net N$111: D55.DO, D56.DI
- new net N$112: D57.CO, D58.CI
- new net N$113: D57.DO, D58.DI
- new net N$114: D58.DO, D59.DI
- new net N$115: D59.CO, D60.CI
- new net N$116: D59.DO, D60.DI
- new net N$117: D58.CO, D59.CI
- new net N$118: D48.CO, D49.CI
- new net N$119: D48.DO, D49.DI
- new net N$12: D5.DO, D6.DI
- new net N$120: D56.DO, D57.DI
- new net N$121: D56.CO, D57.CI
- new net N$124: D20.CO, D21.CI
- new net N$13: D6.CO, D7.CI
- new net N$14: D6.DO, D7.DI
- new net N$15: D7.CO, D8.CI
- new net N$16: D7.DO, D8.DI
- new net N$17: D16.DO, D17.DI
- new net N$18: D20.DO, D21.DI
- new net N$19: D10.CI, D9.CO
- new net N$20: D10.DI, D9.DO
- new net N$21: D10.CO, D11.CI
- new net N$22: D10.DO, D11.DI
- new net N$23: D11.CO, D12.CI
- new net N$24: D11.DO, D12.DI
- new net N$25: D12.CO, D13.CI
- new net N$26: D12.DO, D13.DI
- new net N$27: D13.CO, D14.CI
- new net N$28: D13.DO, D14.DI
- new net N$29: D14.CO, D15.CI
- new net N$30: D14.DO, D15.DI
- new net N$31: D45.CO, D46.CI
- new net N$32: D30.CO, D31.CI
- new net N$33: D8.CO, D9.CI
- new net N$34: D8.DO, D9.DI
- new net N$35: D17.CO, D18.CI
- new net N$36: D17.DO, D18.DI
- new net N$37: D18.CO, D19.CI
- new net N$38: D18.DO, D19.DI
- new net N$39: D19.CO, D20.CI
- new net N$4: D1.CO, D2.CI
- new net N$40: D19.DO, D20.DI
- new net N$41: D30.DO, D31.DI
- new net N$42: D15.CO, D16.CI
- new net N$43: D16.CO, D17.CI
- new net N$44: D21.CO, D22.CI
- new net N$45: D21.DO, D22.DI
- new net N$46: D22.CO, D23.CI
- new net N$47: D22.DO, D23.DI
- new net N$48: D23.CO, D24.CI
- new net N$49: D23.DO, D24.DI
- new net N$5: D1.DO, D2.DI
- new net N$50: D24.CO, D25.CI
- new net N$51: D24.DO, D25.DI
- new net N$52: D25.CO, D26.CI
- new net N$53: D25.DO, D26.DI
- new net N$54: D26.CO, D27.CI
- new net N$55: D26.DO, D27.DI
- new net N$56: D27.CO, D28.CI
- new net N$57: D27.DO, D28.DI
- new net N$58: D29.CO, D30.CI
- new net N$59: D29.DO, D30.DI
- new net N$6: D2.CO, D3.CI
- new net N$60: D15.DO, D16.DI
- new net N$61: D45.DO, D46.DI
- new net N$62: D31.CO, D32.CI
- new net N$63: D31.DO, D32.DI
- new net N$64: D32.CO, D33.CI
- new net N$65: D32.DO, D33.DI
- new net N$66: D33.CO, D34.CI
- new net N$67: D33.DO, D34.DI
- new net N$68: D34.CO, D35.CI
- new net N$69: D34.DO, D35.DI
- new net N$7: D2.DO, D3.DI
- new net N$70: D35.CO, D36.CI
- new net N$71: D35.DO, D36.DI
- new net N$72: D37.CO, D38.CI
- new net N$73: D37.DO, D38.DI
- new net N$74: D38.DO, D39.DI
- new net N$75: D39.CO, D40.CI
- new net N$76: D39.DO, D40.DI
- new net N$77: D38.CO, D39.CI
- new net N$78: D28.CO, D29.CI
- new net N$79: D28.DO, D29.DI
- new net N$8: D3.CO, D4.CI
- new net N$80: D36.DO, D37.DI
- new net N$81: D36.CO, D37.CI
- new net N$82: D40.CO, D41.CI
- new net N$83: D40.DO, D41.DI
- new net N$84: D41.CO, D42.CI
- new net N$85: D41.DO, D42.DI
- new net N$86: D42.CO, D43.CI
- new net N$87: D42.DO, D43.DI
- new net N$88: D43.CO, D44.CI
- new net N$89: D43.DO, D44.DI
- new net N$9: D3.DO, D4.DI
- new net N$90: D44.CO, D45.CI
- new net N$91: D44.DO, D45.DI
- new net N$94: D46.CO, D47.CI
- new net N$95: D46.DO, D47.DI
- new net N$96: D47.CO, D48.CI
- new net N$97: D47.DO, D48.DI
- new net N$98: D49.CO, D50.CI
- new net N$99: D49.DO, D50.DI
- net 5V: now also D1.VCC, D10.VCC, D11.VCC, D12.VCC, D13.VCC, D14.VCC, D15.VCC, D16.VCC, D17.VCC, D18.VCC, D19.VCC, D2.VCC, D20.VCC, D21.VCC, D22.VCC, D23.VCC, D24.VCC, D25.VCC, D26.VCC, D27.VCC, D28.VCC, D29.VCC, D3.VCC, D30.VCC, D31.VCC, D32.VCC, D33.VCC, D34.VCC, D35.VCC, D36.VCC, D37.VCC, D38.VCC, D39.VCC, D4.VCC, D40.VCC, D41.VCC, D42.VCC, D43.VCC, D44.VCC, D45.VCC, D46.VCC, D47.VCC, D48.VCC, D49.VCC, D5.VCC, D50.VCC, D51.VCC, D52.VCC, D53.VCC, D54.VCC, D55.VCC, D56.VCC, D57.VCC, D58.VCC, D59.VCC, D6.VCC, D60.VCC, D7.VCC, D8.VCC, D9.VCC
- net CI: now also D1.CI
- net CO: now also D60.CO
- net DI: now also D1.DI
- net DO: now also D60.DO
- net GND: now also D1.GND, D10.GND, D11.GND, D12.GND, D13.GND, D14.GND, D15.GND, D16.GND, D17.GND, D18.GND, D19.GND, D2.GND, D20.GND, D21.GND, D22.GND, D23.GND, D24.GND, D25.GND, D26.GND, D27.GND, D28.GND, D29.GND, D3.GND, D30.GND, D31.GND, D32.GND, D33.GND, D34.GND, D35.GND, D36.GND, D37.GND, D38.GND, D39.GND, D4.GND, D40.GND, D41.GND, D42.GND, D43.GND, D44.GND, D45.GND, D46.GND, D47.GND, D48.GND, D49.GND, D5.GND, D50.GND, D51.GND, D52.GND, D53.GND, D54.GND, D55.GND, D56.GND, D57.GND, D58.GND, D59.GND, D6.GND, D60.GND, D7.GND, D8.GND, D9.GND
Other:
- note added: "LED's"
- note added: "Vin: 3.0V-5.5V"
