File: DesignVFD-Ring.sch (EAGLE design)
At the start: 32 parts, among them IC1 LMR64010XMF/NOPB, IC2 LM340S-05, U1 MAX6920AWP+, U2 LM1084IS-5.0, U3 TPS76325DBVT

Commit message: IVL complete
Connections:
- removed net N$10: U$2.MIDDLE, U1.OUT3
- removed net N$11: U$2.LOWERLEFT, U1.OUT4
- removed net N$12: U$2.LOWERRIGHT, U1.OUT5
- removed net N$13: U$2.LOWER, U1.OUT6
- removed net N$14: U$2.GRID1, U1.OUT7
- removed net N$15: U$2.GRID2, U1.OUT8
- removed net N$16: U$2.GRID4, U1.OUT9
- removed net N$17: U$2.GRID5, U1.OUT10
- removed net N$5: U$2.TOPSEGMENT, U1.OUT0
- removed net N$8: U$2.TOPLEFT, U1.OUT1
- removed net N$9: U$2.TOPRIGHT, U1.OUT2
- new net BDOT: U$2.BOTTOMDOT
- new net G1: U$2.GRID1, U1.OUT5
- new net G2: U$2.GRID2, U1.OUT2
- new net G3: U$2.GRID3
- new net G4: U$2.GRID4, U1.OUT11
- new net G5: U$2.GRID5, U1.OUT7
- new net LOW: U$2.LOWER, U1.OUT0
- new net LOW_L: U$2.LOWERLEFT, U1.OUT3
- new net LOW_R: U$2.LOWERRIGHT, U1.OUT1
- new net MID: U$2.MIDDLE, U1.OUT4
- new net NC: U1.OUT6
- new net TDOT: U$2.TOPDOT
- new net TOP: U$2.TOPSEGMENT, U1.OUT8
- new net TOP_L: U$2.TOPLEFT, U1.OUT9
- new net TOP_R: U$2.TOPRIGHT, U1.OUT10

Commit message: Passed ERC and DRC!
Parts:
- added JP4: (no value), pinhead:PINHD-1X1
Connections:
- net GND: now also JP4.1
Changed lines of the file:
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@@
 <part name="U$4" library="FormE" deviceset="LUMINI3" device=""/>
 <part name="JP3" library="pinhead" library_urn="urn:adsk.eagle:library:325" deviceset="PINHD-1X1" device="" package3d_urn="urn:adsk.eagle:package:22485/2"/>
+<part name="JP4" library="pinhead" library_urn="urn:adsk.eagle:library:325" deviceset="PINHD-1X1" device="" package3d_urn="urn:adsk.eagle:package:22485/2"/>
 </parts>
 <sheets>
@@
 <attribute name="VALUE" x="-3.81" y="330.2" size="1.778" layer="96" rot="MR0"/>
 </instance>
+<instance part="JP4" gate="G$1" x="-10.16" y="327.66" smashed="yes" rot="MR0">
+<attribute name="NAME" x="-3.81" y="330.835" size="1.778" layer="95" rot="MR0"/>
+<attribute name="VALUE" x="-3.81" y="322.58" size="1.778" layer="96" rot="MR0"/>
+</instance>
 </instances>
 <busses>
@@
 <wire x1="25.4" y1="327.66" x2="38.1" y2="327.66" width="0.1524" layer="91"/>
 <junction x="25.4" y="327.66"/>
+<pinref part="JP4" gate="G$1" pin="1"/>
+<wire x1="-7.62" y1="327.66" x2="10.16" y2="327.66" width="0.1524" layer="91"/>
+<junction x="10.16" y="327.66"/>
 </segment>
 <segment>
@@
 </sheet>
 </sheets>
+<errors>
+</errors>
 </schematic>
 </drawing>

Commit message: added aesthetic capacitor
Parts:
- added C10: (no value), rcl:C-US025-050X050
Connections:
- net +12V: now also C10.1
- net GND: now also C10.2
Changed lines of the file:
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@@
 <part name="JP3" library="pinhead" library_urn="urn:adsk.eagle:library:325" deviceset="PINHD-1X1" device="" package3d_urn="urn:adsk.eagle:package:22485/2"/>
 <part name="JP4" library="pinhead" library_urn="urn:adsk.eagle:library:325" deviceset="PINHD-1X1" device="" package3d_urn="urn:adsk.eagle:package:22485/2"/>
+<part name="C10" library="rcl" library_urn="urn:adsk.eagle:library:334" deviceset="C-US" device="025-050X050" package3d_urn="urn:adsk.eagle:package:23633/1"/>
+<part name="GND12" library="supply1" library_urn="urn:adsk.eagle:library:371" deviceset="GND" device=""/>
 </parts>
 <sheets>
@@
 <attribute name="VALUE" x="-3.81" y="322.58" size="1.778" layer="96" rot="MR0"/>
 </instance>
+<instance part="C10" gate="G$1" x="-12.7" y="200.66" smashed="yes">
+<attribute name="NAME" x="-11.684" y="201.295" size="1.778" layer="95"/>
+<attribute name="VALUE" x="-11.684" y="196.469" size="1.778" layer="96"/>
+</instance>
+<instance part="GND12" gate="1" x="-12.7" y="193.04" smashed="yes">
+<attribute name="VALUE" x="-15.24" y="190.5" size="1.778" layer="96"/>
+</instance>
 </instances>
 <busses>
@@
 <wire x1="119.38" y1="50.8" x2="116.84" y2="50.8" width="0.1524" layer="91"/>
 </segment>
+<segment>
+<pinref part="C10" gate="G$1" pin="2"/>
+<pinref part="GND12" gate="1" pin="GND"/>
+</segment>
 </net>
 <net name="T_IGN_INPUT" class="0">
@@
 <pinref part="IC1" gate="G$1" pin="!SHDN"/>
 <wire x1="5.08" y1="203.2" x2="5.08" y2="185.42" width="0.1524" layer="91"/>
-</segment>
-</net>
+<pinref part="C10" gate="G$1" pin="1"/>
+<wire x1="-12.7" y1="203.2" x2="5.08" y2="203.2" width="0.1524" layer="91"/>
+<junction x="5.08" y="203.2"/>
+</segment>
+</net>

Commit message: created and added logo, removed board markings
Parts:
- U$1: value 10uF -> 10uH
Changed lines of the file:
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@@
 <part name="U1" library="MAX6920AWP_" deviceset="MAX6920AWP+" device=""/>
 <part name="D1" library="diode" library_urn="urn:adsk.eagle:library:210" deviceset="MBR0520LT" device="" package3d_urn="urn:adsk.eagle:package:43420/1"/>
-<part name="U$1" library="FormE" deviceset="732-1416-ND" device="732-1416-ND" value="10uF"/>
+<part name="U$1" library="FormE" deviceset="732-1416-ND" device="732-1416-ND" value="10uH"/>
 <part name="U2" library="LM1084IS-5.0" deviceset="LM1084IS-5.0" device=""/>
 <part name="U3" library="TPS76325DBVT" deviceset="TPS76325DBVT" device=""/>
